File: Digital.kicad_sch (KiCad schematic)
At the start: 12 parts, among them J5 SAI, J6 Vol, U3 PCM3060, U5 PGA2310

Commit message: Addition of a second relay to enable true hardware bypass
Other:
- title: OSCAR Audio 01 V2 -> OSCAR Audio 01 V2.1
