File: OSCAR_Audio.kicad_sch (KiCad schematic)
At the start: 0 parts

Commit message: Invert output summing stage to maintain correct phase
Other:
- title: OSCAR Audio 1.0 -> OSCAR Audio 01 V2
Changed lines of the file:
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@@
 	(paper "A4")
 	(title_block
-		(title "OSCAR Audio 1.0")
+		(title "OSCAR Audio 01 V2")
 		(date "2025-05-30")
-		(rev "2")
+		(rev "2.1")
 		(company "DAD Design")
 	)
