File: OSCAR_Audio.kicad_sch (KiCad schematic)
At the start: 0 parts

Commit message: Addition of a second relay to enable true hardware bypass
Other:
- title: OSCAR Audio 01 V2 -> OSCAR Audio 01 V2.1
Changed lines of the file:
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@@
 (kicad_sch
-	(version 20250114)
+	(version 20260306)
 	(generator "eeschema")
-	(generator_version "9.0")
+	(generator_version "10.0")
 	(paper "A4")
 	(title_block
-		(title "OSCAR Audio 01 V2")
+		(title "OSCAR Audio 01 V2.1")
 		(date "2025-05-30")
-		(rev "2.1")
+		(rev "1.0")
 		(company "DAD Design")
 	)
@@
 		)
 		(fill
-			(color 0 0 0 0.0000)
+			(color 0 0 0 0)
 		)
 		(property "Sheetname" "Digital"
 			(at 160.02 31.0384 0)
+			(show_name no)
+			(do_not_autoplace no)
 			(effects
 				(font
@@
 		(property "Sheetfile" "Digital.kicad_sch"
 			(at 160.02 81.8646 0)
+			(show_name no)
+			(do_not_autoplace no)
 			(effects
 				(font
@@
 		)
 		(fill
-			(color 0 0 0 0.0000)
+			(color 0 0 0 0)
 		)
 		(property "Sheetname" "Alim"
 			(at 50.8 100.8884 0)
+			(show_name no)
+			(do_not_autoplace no)
 			(effects
 				(font
@@
 		(property "Sheetfile" "Alim.kicad_sch"
 			(at 50.8 150.4446 0)
+			(show_name no)
+			(do_not_autoplace no)
 			(effects
 				(font
@@
 		)
 		(fill
-			(color 0 0 0 0.0000)
+			(color 0 0 0 0)
 		)
 		(property "Sheetname" "Analog"
 			(at 50.8 32.3084 0)
+			(show_name no)
+			(do_not_autoplace no)
 			(effects
 				(font
@@
 		(property "Sheetfile" "Analog.kicad_sch"
 			(at 50.8 84.4046 0)
+			(show_name no)
+			(do_not_autoplace no)
 			(effects
 				(font
