File: Alim.kicad_sch (KiCad schematic)
At the start: 48 parts, among them J7 +12V, J8 +12V, U1 OPA1642, U2 OPA1644, U3 PCM3060, U4 NE5532, U5 PGA2310, U6 LM317_SOT-223, U7 LM337_SOT223, U8 L78L05_SOT89

Commit message: Addition of a second relay to enable true hardware bypass
Parts:
- FB2, FB4: footprint Inductor_SMD:L_0805_2012Metric_Pad1.15x1.40mm_HandSolder -> Inductor_SMD:L_0805_2012Metric_Pad1.05x1.20mm_HandSolder
Other:
- title: OSCAR Audio 01 V2 -> OSCAR Audio 01 V2.1
