File: Analog.kicad_sch (KiCad schematic)
At the start: 72 parts, among them J1 InL, J2 InR, J3 OutR, J4 OutL, J9 ByPass, K1 G6K-2F-Y, U1 OPA1642, U2 OPA1644, U3 PCM3060, U4 NE5532, U5 PGA2310

Commit message: Addition of a second relay to enable true hardware bypass
Parts:
- added D2: 1N4148W, Diode_SMD:D_SOD-123, symbol Diode:1N4148W
- added K2: G6K-2F-Y, Relay_SMD:Relay_DPDT_Omron_G6K-2F-Y, symbol Relay:G6K-2
- R19, R22, R30, R33: value 10k -> 22k
Connections:
- net +R5V: now also D2.1 (K), K2.1
- net R0V: now also D2.2 (A), K2.8
- net at J3.T: now also K2.3; no longer K1.3
- net at J4.T: now also K2.6; no longer K1.6
- net at C19.1, R34.1: now also K2.5; no longer K1.5
- net at C15.1, R24.1: now also K2.4; no longer K1.4
- net at J1.T, J2.TN: now also K1.6; no longer C2.1, K1.7
- new net: K1.2, K2.2
- new net: K1.7, K2.7
- new net: J2.T, K1.3
- new net: C9.1, K1.4
- new net: C2.1, K1.5
Other:
- title: OSCAR Audio 01 V2 -> OSCAR Audio 01 V2.1
- moved on the sheet: C1, C10, C11, C12, C15, C19, C2, C3, C4, C5, C6, C7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
