File: OSCAR_Audio.kicad_pcb (KiCad board)
At the start: 2 copper layers, 91 x 87.1 mm, 127 parts, among them J1 InL, J2 InR, J3 OutR, J4 OutL, J5 SAI, J6 Vol, J7 +12V, J8 +12V, J9 ByPass, K1 G6K-2F-Y, U1 OPA1642, U2 OPA1644, U3 PCM3060, U4 NE5532, U5 PGA2310, U6 LM317_SOT-223, U7 LM337_SOT223, U8 L78L05_SOT89

Commit message: Addition of a second relay to enable true hardware bypass
Parts:
- added D2: 1N4148W, Diode_SMD:D_SOD-123, F.Cu at (120.4, 48.7)
- added K2: G6K-2F-Y, Relay_SMD:Relay_DPDT_Omron_G6K-2F-Y, F.Cu at (123.8, 56.5)
- D1: moved to F.Cu
- FB2, FB4: footprint Inductor_SMD:L_0805_2012Metric_Pad1.15x1.40mm_HandSolder -> Inductor_SMD:L_0805_2012Metric_Pad1.05x1.20mm_HandSolder
- R19, R22, R30, R33: value 10k -> 22k
- moved D1 36.8 mm to (144.2, 48.7)
- moved K1 23.0 mm to (146.0, 55.6), turned to 0 degrees
- moved C19 5.15 mm to (127.3, 65.1)
- moved R34 5.02 mm to (124.4, 65.1)
- moved C15 3.13 mm to (150.9, 66.2), turned to 0 degrees
- moved R24 2.82 mm to (143.7, 65.1), turned to 180 degrees
- moved C2 1.16 mm to (173.2, 63.2), turned to 0 degrees
- moved C9 0.38 mm to (195.3, 62.3), turned to 0 degrees
Connections:
- J1 pad T: Net-(C2-Pad1) -> Net-(J1-PadT)
- J2 pad T: Net-(C9-Pad1) -> Net-(J2-PadT)
- J2 pad TN: Net-(C2-Pad1) -> Net-(J1-PadT)
- K1 pad 2: Net-(C9-Pad1) -> Net-(K1-Pad2)
- K1 pad 3: Net-(J3-PadT) -> Net-(J2-PadT)
- K1 pad 4: Net-(C15-Pad1) -> Net-(C9-Pad1)
- K1 pad 5: Net-(C19-Pad1) -> Net-(C2-Pad1)
- K1 pad 6: Net-(J4-PadT) -> Net-(J1-PadT)
- K1 pad 7: Net-(C2-Pad1) -> Net-(K1-Pad7)
Routing:
- net Net-(J2-PadT): track 0.00 -> 68.3 mm, vias 0 -> 2
- net Net-(C2-Pad1): track 67.5 -> 24.7 mm, vias 1 -> 2
- net /Analog/R0V: track 25.7 -> 64.7 mm, vias 1 -> 2
- net Net-(J1-PadT): track 0.00 -> 36.8 mm, vias 0 -> 1
- net Net-(K1-Pad7): track 0.00 -> 29.2 mm, vias 0 -> 2
- net Net-(C9-Pad1): track 92.6 -> 65.8 mm, vias 1 -> 2
- net Net-(K1-Pad2): track 0.00 -> 24.2 mm
- net /Analog/+R5V: track 35.0 -> 52.9 mm, vias 1 -> 0
- net Net-(U1B-+): track 32.1 -> 41.3 mm
- net Net-(J4-PadT): track 13.7 -> 6.62 mm
- net Net-(C19-Pad2): track 96.7 -> 90.4 mm
- net Net-(C15-Pad2): track 80.0 -> 76.2 mm
- net Net-(C19-Pad1): track 9.60 -> 6.14 mm
- net Net-(J3-PadT): track 39.0 -> 35.6 mm, vias 0 -> 1
- net GNDA: track 198.4 -> 195.2 mm, vias 47 -> 54
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Other:
- board text added: "OSCAR-AUDIO-01 V2.2"
- board text removed: "OSCAR-AUDIO-01 V2.1"
